File: PCB-SMD/ToneGenerator.kicad_pcb (KiCad board)
At the start: 2 copper layers, 30 x 80.8 mm, 37 parts, among them CN100 IN, IC1 AMS1117-5V, J100 Con-Rotatif-1X12, Q1 BS170-L, Q2 CJ2310

Commit message: PCB Update
Parts:
- IC1: value AMS1117-5V -> AMS1117
- moved REF** 22.4 mm to (145.3, 123.4), turned to -90 degrees
- moved REF** 1.37 mm to (142.0, 82.8)
Connections:
- CN100 pad 1: Net-(CN100-Pin_1) -> GND
- CN100 pad 2: Net-(CN100-Pin_2) -> /SIN0
- CN100 pad 3: Net-(CN100-Pin_3) -> +5V
- J100 pad 1: Net-(CN100-Pin_3) -> +5V
- J100 pad 12: Net-(CN100-Pin_1) -> GND
- R1 pad 2: Net-(SIN0-KL) -> /SIN0
- R100 pad 2: Net-(CN100-Pin_2) -> /SIN0
- R101 pad 1: Net-(CN100-Pin_3) -> +5V
- R102 pad 1: Net-(CN100-Pin_1) -> GND
- SIN0 pad 1: Net-(SIN0-KL) -> /SIN0
Routing:
- net /SIN0: track 0.00 -> 117.0 mm
- net +5V: track 24.5 -> 72.5 mm, vias 1 -> 2
- net GND: track 14.3 -> 33.2 mm
- net Net-(SIN0-KL): track 12.3 -> 0.00 mm
- net Net-(CN100-Pin_3): track 8.95 -> 0.00 mm
- net Net-(CN100-Pin_1): track 8.66 -> 0.00 mm
- net Net-(CN100-Pin_2): track 7.65 -> 0.00 mm
Other:
- board text added: "https://github.com/alcarbure/ToneGenerator-for-NEC"
- board text removed: "S202419-1"
