File: PCB-SMD/ToneGenerator.kicad_sch (KiCad schematic)
At the start: 35 parts, among them CN100 IN, IC1 AMS1117, J100 Con-Rotatif-1X12, Q1 BS170-L, Q2 CJ2310

Commit message: PCB Update
Connections:
- net +5V: now also CN100.3 (Pin_3), J100.1, R101.1
- net GND: now also CN100.1 (Pin_1), J100.12, R102.1
- net SIN0: now reaches R1.2, SIN0.1 (KL)
- net SIN0: now also CN100.2 (Pin_2), R100.2
Other:
- note added: "1"
- note added: "2"
- note added: "3"
- moved on the sheet: ARD1B, C2, D1, IC1, JP1, S+0, S-0, SIN0
